File: Hardware/SparkFun_GNSS_LG580P.kicad_pcb (KiCad board)
At the start: 4 copper layers, 50.8 x 43.2 mm, 159 parts, among them J1 USB_C_Receptacle, J10 Conn_01x06, J2 Conn_01x06, J3 SMA_Edge, J4 Qwiic_RA, J5 SMA_Edge, J6 Conn_01x09, J7 Qwiic_RA, J8 JST_Locking_4, J9 I2C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

Commit message: Post design review changes
Parts:
- removed kibuzzard-6797D26F: G***, kibuzzard-6797D26F
- removed kibuzzard-6797D27F: G***, kibuzzard-6797D27F
- added TP2: 1.0mm, SparkFun-Connector:TestPoint-1.0mm, B.Cu at (172.6, 78.6)
- added TP3: 1.0mm, SparkFun-Connector:TestPoint-1.0mm, B.Cu at (179.9, 78.6)
- added kibuzzard-67A3F35B: G***, kibuzzard-67A3F35B, B.Cu at (159.4, 113.3)
- added kibuzzard-67A3F366: G***, kibuzzard-67A3F366, F.Cu at (159.4, 113.3)
- J4, J7: footprint SparkFun-Connector:JST_SMD_1.0mm-4_RA -> SparkFun-Connector:JST_SMD_1.0mm-4_Black
- JP1: value BT-VCC -> ~
- JP2: value PWR -> ~
- JP3: value PPS -> ~
- JP4: value VSEL -> ~
- JP5: value RTK -> ~
- JP6: value HEAD -> ~
- JP8: value PVT -> ~
- R10: value 1k -> 330
- moved kibuzzard-6797CEC8 0.79 mm to (179.9, 105.4) (x2)
- moved kibuzzard-6797CECC 0.79 mm to (179.9, 86.4) (x2)
- moved kibuzzard-6797CEB8 0.63 mm to (180.0, 95.9)
- moved J3 0.16 mm to (183.7, 105.4)
- moved J5 0.16 mm to (183.7, 86.4)
Routing:
- net TXD3: track 39.6 -> 44.2 mm, vias 2 -> 3
- net Net-(J8-Pin_3): track 5.88 -> 8.73 mm, vias 0 -> 1
- net GND: track 4.80 -> 7.09 mm, vias 155 -> 163
