File: Hardware/SparkFun_GNSS_LG580P.kicad_sch (KiCad schematic)
At the start: 76 parts, among them J1 USB_C_Receptacle, J10 Conn_01x06, J2 Conn_01x06, J3 SMA_Edge, J4 Qwiic_RA, J5 SMA_Edge, J6 Conn_01x09, J7 Qwiic_RA, J8 JST_Locking_4, J9 I2C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

Commit message: Post design review changes
Parts:
- added TP2, TP3: 1.0mm, SparkFun-Connector:TestPoint-1.0mm, symbol SparkFun-Connector:TestPoint_1.0mm
- J4, J7: footprint SparkFun-Connector:JST_SMD_1.0mm-4_RA -> SparkFun-Connector:JST_SMD_1.0mm-4_Black
- JP1: value BT-VCC -> ~
- JP2: value PWR -> ~
- JP3: value PPS -> ~
- JP4: value VSEL -> ~
- JP5: value RTK -> ~
- JP6: value HEAD -> ~
- JP8: value PVT -> ~
- R10: value 1k -> 330; symbol SparkFun-Resistor:1k_0603 -> SparkFun-Resistor:330_0603; PROD_ID RES-07856 -> RES-00818
Connections:
- net TXD3: now also TP3.1
- net at J8.3 (Pin_3), R8.1: now also TP2.1
Other:
- note added: "Coplanar 50Ω Waveguide Calculation: Copper Thickness (1oz): 1.4mil/0.035mm Board thickness: 1.6mm Dielectric thickness (layer 1 to 2): 0.2mm Er: 4.6 Polygon Isolation: 8mil/0.2032mm RF Trace Width: 13.74mil/0.349mm https://chemandy.com/calculators/coplanar-waveguide-with-ground-calculator.htm"
- note removed: "Coplanar Waveguide Calculation: Copper Thickness (1oz): 1.4mil/0.035mm Board thickness: 1.6mm Dielectric thickness (layer 1 to 2): 0.2mm Er: 4.6 Polygon Isolation: 8mil/0.2032mm RF Trace Width: 13.74mil/0.349mm https://chemandy.com/calculators/coplanar-waveguide-with-ground-calculator.htm"
- moved on the sheet: R8
Changed lines of the file:
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@@
 	)
 	(junction
+		(at 156.21 227.33)
+		(diameter 0)
+		(color 0 0 0 0)
+	)
+	(junction
 		(at 167.64 63.5)
 		(diameter 0)
@@
 		(color 0 0 0 0)
 	)
+	(junction
+		(at 152.4 224.79)
+		(diameter 0)
+		(color 0 0 0 0)
+	)
 	(no_connect
 		(at 101.6 52.07)
@@
 	(wire
 		(pts
+			(xy 156.21 227.33) (xy 161.29 227.33)
+		)
+		(stroke
+			(width 0)
+			(type default)
+		)
+	)
+	(wire
+		(pts
 			(xy 120.65 227.33) (xy 123.19 227.33)
 		)
@@
 	(wire
 		(pts
-			(xy 152.4 227.33) (xy 153.67 227.33)
+			(xy 152.4 224.79) (xy 161.29 224.79)
 		)
 		(stroke
@@
 	(wire
 		(pts
-			(xy 158.75 227.33) (xy 161.29 227.33)
+			(xy 153.67 227.33) (xy 156.21 227.33)
 		)
 		(stroke
@@
 	(wire
 		(pts
-			(xy 160.02 224.79) (xy 161.29 224.79)
+			(xy 147.32 224.79) (xy 152.4 224.79)
 		)
 		(stroke
@@
 	(wire
 		(pts
+			(xy 147.32 227.33) (xy 148.59 227.33)
+		)
+		(stroke
+			(width 0)
+			(type default)
+		)
+	)
+	(wire
+		(pts
 			(xy 341.63 66.04) (xy 340.36 66.04)
 		)
@@
 	(wire
 		(pts
+			(xy 156.21 227.33) (xy 156.21 228.6)
+		)
+		(stroke
+			(width 0)
+			(type default)
+		)
+	)
+	(wire
+		(pts
 			(xy 389.89 158.75) (xy 394.97 158.75)
 		)
@@
 	(wire
 		(pts
+			(xy 152.4 223.52) (xy 152.4 224.79)
+		)
+		(stroke
+			(width 0)
+			(type default)
+		)
+	)
+	(wire
+		(pts
 			(xy 337.82 158.75) (xy 337.82 161.29)
 		)
@@
 		)
 	)
-	(text "Coplanar Waveguide Calculation:\nCopper Thickness (1oz): 1.4mil/0.035mm\nBoard thickness: 1.6mm\nDielectric thickness (layer 1 to 2): 0.2mm\nEr: 4.6\nPolygon Isolation: 8mil/0.2032mm\nRF Trace Width: 13.74mil/0.349mm\nhttps://chemandy.com/calculators/coplanar-waveguide-with-ground-calculator.htm"
+	(text "Coplanar 50Ω Waveguide Calculation:\nCopper Thickness (1oz): 1.4mil/0.035mm\nBoard thickness: 1.6mm\nDielectric thickness (layer 1 to 2): 0.2mm\nEr: 4.6\nPolygon Isolation: 8mil/0.2032mm\nRF Trace Width: 13.74mil/0.349mm\nhttps://chemandy.com/calculators/coplanar-waveguide-with-ground-calculator.htm"
 		(exclude_from_sim no)
 		(at 328.93 196.85 0)
@@
 	(global_label "RXD3"
 		(shape input)
-		(at 152.4 227.33 180)
+		(at 147.32 227.33 180)
 		(fields_autoplaced yes)
 		(effects
@@
 		)
 		(property "Intersheetrefs" "${INTERSHEET_REFS}"
-			(at 144.4558 227.33 0)
+			(at 139.3758 227.33 0)
 			(effects
 				(font
@@
 	(global_label "TXD3"
 		(shape input)
-		(at 160.02 224.79 180)
+		(at 147.32 224.79 180)
 		(fields_autoplaced yes)
 		(effects
@@
 		)
 		(property "Intersheetrefs" "${INTERSHEET_REFS}"
-			(at 152.3782 224.79 0)
+			(at 139.6782 224.79 0)
 			(effects
 				(font
@@
 	)
 	(symbol
+		(lib_id "SparkFun-Connector:TestPoint_1.0mm")
+		(at 152.4 223.52 0)
+		(unit 1)
+		(exclude_from_sim no)
+		(in_bom yes)
+		(on_board yes)
+		(dnp no)
+		(fields_autoplaced yes)
+		(property "Reference" "TP3"
+			(at 152.4 218.44 0)
+			(do_not_autoplace yes)
+			(effects
+				(font
+					(size 1.27 1.27)
+				)
+			)
+		)
+		(property "Value" "1.0mm"
+			(at 152.4 227.33 0)
+			(effects
+				(font
+					(size 1.27 1.27)
+				)
+				(hide yes)
+			)
+		)
+		(property "Footprint" "SparkFun-Connector:TestPoint-1.0mm"
+			(at 152.4 229.87 0)
+			(effects
+				(font
+					(size 1.27 1.27)
+				)
+				(hide yes)
+			)
+		)
+		(property "Datasheet" "~"
+			(at 152.4 231.14 0)
+			(effects
+				(font
+					(size 1.27 1.27)
+				)
+				(hide yes)
+			)
+		)
+		(property "Description" "Test Point"
+			(at 152.4 233.68 0)
+			(effects
+				(font
+					(size 1.27 1.27)
+				)
+				(hide yes)
+			)
+		)
+		(pin "1"
+		)
+		(instances
+			(project ""
+				(path "/e3dd3ae4-244d-4cba-9cca-5d2abf83f29a"
+					(reference "TP3")
+					(unit 1)
+				)
+			)
+		)
+	)
+	(symbol
 		(lib_id "SparkFun-RF:SMA_EdgeMount")
 		(at 317.5 142.24 0)
@@
 			)
 		)
-		(property "Value" "RTK"
+		(property "Value" "~"
 			(at 256.54 222.25 0)
 			(effects
@@
 	)
 	(symbol
-		(lib_id "SparkFun-Resistor:1k_0603")
+		(lib_id "SparkFun-Resistor:330_0603")
 		(at 264.16 228.6 90)
 		(unit 1)
@@
 			)
 		)
-		(property "Value" "1k"
+		(property "Value" "330"
 			(at 266.7 229.8699 90)
 			(effects
@@
 		)
 		(property "Footprint" "SparkFun-Resistor:R_0603_1608Metric"
-			(at 264.16 224.028 90)
+			(at 268.732 228.6 0)
 			(effects
 				(font
@@
 		)
 		(property "Datasheet" "https://www.vishay.com/docs/20035/dcrcwe3.pdf"
-			(at 264.16 228.6 0)
+			(at 273.05 228.6 0)
 			(effects
 				(font
@@
 		)
 		(property "Description" "Resistor"
-			(at 264.16 228.6 0)
+			(at 275.59 228.6 0)
 			(effects
 				(font
@@
 			)
 		)
-		(property "PROD_ID" "RES-07856"
-			(at 264.16 221.742 90)
+		(property "PROD_ID" "RES-00818"
+			(at 271.018 228.6 0)
 			(effects
 				(font
@@
 			)
 		)
-		(property "Value" "VSEL"
+		(property "Value" "~"
 			(at 160.02 215.646 0)
 			(effects
@@
 			)
 		)
-		(property "Footprint" "SparkFun-Connector:JST_SMD_1.0mm-4_RA"
+		(property "Footprint" "SparkFun-Connector:JST_SMD_1.0mm-4_Black"
 			(at 72.39 153.67 0)
 			(effects
@@
 			)
 		)
-		(property "Value" "PWR"
+		(property "Value" "~"
 			(at 236.22 222.25 0)
 			(effects
@@
 	(symbol
 		(lib_id "SparkFun-Resistor:1k_0603")
-		(at 156.21 227.33 180)
+		(at 151.13 227.33 180)
 		(unit 1)
 		(exclude_from_sim no)
@@
 		(on_board yes)
 		(dnp no)
-		(fields_autoplaced yes)
 		(property "Reference" "R8"
-			(at 156.21 231.14 0)
+			(at 151.13 229.87 0)
 			(effects
 				(font
@@
 		)
 		(property "Value" "1k"
-			(at 156.21 233.68 0)
+			(at 151.13 232.41 0)
 			(effects
 				(font
@@
 		)
 		(property "Footprint" "SparkFun-Resistor:R_0603_1608Metric"
-			(at 151.638 227.33 90)
+			(at 146.558 227.33 90)
 			(effects
 				(font
@@
 		)
 		(property "Datasheet" "https://www.vishay.com/docs/20035/dcrcwe3.pdf"
-			(at 147.32 226.06 90)
+			(at 142.24 226.06 90)
 			(effects
 				(font
@@
 		)
 		(property "Description" "Resistor"
-			(at 156.21 227.33 0)
+			(at 151.13 227.33 0)
 			(effects
 				(font
@@
 		)
 		(property "PROD_ID" "RES-07856"
-			(at 149.352 227.33 90)
+			(at 144.272 227.33 90)
 			(effects
 				(font
@@
 	)
 	(symbol
+		(lib_id "SparkFun-Connector:TestPoint_1.0mm")
+		(at 156.21 228.6 180)
+		(unit 1)
+		(exclude_from_sim no)
+		(in_bom yes)
+		(on_board yes)
+		(dnp no)
+		(fields_autoplaced yes)
+		(property "Reference" "TP2"
+			(at 156.21 233.68 0)
+			(do_not_autoplace yes)
+			(effects
+				(font
+					(size 1.27 1.27)
+				)
+			)
+		)
+		(property "Value" "1.0mm"
+			(at 156.21 224.79 0)
+			(effects
+				(font
+					(size 1.27 1.27)
+				)
+				(hide yes)
+			)
+		)
+		(property "Footprint" "SparkFun-Connector:TestPoint-1.0mm"
+			(at 156.21 222.25 0)
+			(effects
+				(font
+					(size 1.27 1.27)
+				)
+				(hide yes)
+			)
+		)
+		(property "Datasheet" "~"
+			(at 156.21 220.98 0)
+			(effects
+				(font
+					(size 1.27 1.27)
+				)
+				(hide yes)
+			)
+		)
+		(property "Description" "Test Point"
+			(at 156.21 218.44 0)
+			(effects
+				(font
+					(size 1.27 1.27)
+				)
+				(hide yes)
+			)
+		)
+		(pin "1"
+		)
+		(instances
+			(project "SparkFun_GNSS_LG580P"
+				(path "/e3dd3ae4-244d-4cba-9cca-5d2abf83f29a"
+					(reference "TP2")
+					(unit 1)
+				)
+			)
+		)
+	)
+	(symbol
 		(lib_id "SparkFun-PowerSymbol:3.3V")
 		(at 233.68 218.44 0)
@@
 			)
 		)
-		(property "Value" "BT-VCC"
+		(property "Value" "~"
 			(at 123.19 218.44 90)
 			(effects
@@
 			)
 		)
-		(property "Value" "HEAD"
+		(property "Value" "~"
 			(at 266.7 222.25 0)
 			(effects
@@
 			)
 		)
-		(property "Value" "PVT"
+		(property "Value" "~"
 			(at 276.86 222.25 0)
 			(effects
@@
 			)
 		)
-		(property "Footprint" "SparkFun-Connector:JST_SMD_1.0mm-4_RA"
+		(property "Footprint" "SparkFun-Connector:JST_SMD_1.0mm-4_Black"
 			(at 104.14 153.67 0)
 			(effects
@@
 			)
 		)
-		(property "Value" "PPS"
+		(property "Value" "~"
 			(at 246.38 222.25 0)
 			(effects

Commit message: Add panelized files
Parts:
- removed D6, D7: PESD0603-240, SparkFun-Capacitor:C_0603_1608Metric, symbol SparkFun-DiscreteSemi:D_TVS_0603
- added D11: DF5A5.6LFU, SparkFun-Semiconductor-Standard:SOT-353, symbol SparkFun-DiscreteSemi:D_TVS_ESD_4_HS_3.3V
Connections:
- net 3.3V: now also D11.1 (K1)
- net GND: now also D11.2 (A)
- net V_BCKP: now also D11.5 (K4)
Other:
- moved on the sheet: C1, C2, C5, C8, R9, U2

Commit message: Update to KiCad v9
Changed lines of the file:
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@@
 (kicad_sch
-	(version 20231120)
+	(version 20250114)
 	(generator "eeschema")
-	(generator_version "8.0")
+	(generator_version "9.0")
 	(paper "USLedger")
 	(title_block
@@
 		(comment 1 "Designed by: N. Seidle")
 	)
+	(text "I²C Connectors"
+		(exclude_from_sim no)
+		(at 105.41 124.46 0)
+		(effects
+			(font
+				(size 3 3)
+			)
+		)
+	)
+	(text "Generally speaking the ports are used as follows:\nUART1 - Configure in and NMEA output over USB\nUART2 - RTCM correction input and NMEA output over Bluetooth\nUART3 - NMEA output to embedded system"
+		(exclude_from_sim no)
+		(at 116.84 254 0)
+		(effects
+			(font
+				(size 1.5 1.5)
+			)
+			(justify left)
+		)
+	)
+	(text "Reset has\ninternal pull-up."
+		(exclude_from_sim no)
+		(at 289.56 41.91 0)
+		(effects
+			(font
+				(size 1.5 1.5)
+			)
+		)
+	)
+	(text "I²C interface not yet supported.\nSupport coming in future firmware release."
+		(exclude_from_sim no)
+		(at 101.6 163.83 0)
+		(effects
+			(font
+				(size 3 3)
+			)
+		)
+	)
+	(text "Coplanar 50Ω Waveguide Calculation:\nCopper Thickness (1oz): 1.4mil/0.035mm\nBoard thickness: 1.6mm\nDielectric thickness (layer 1 to 2): 0.2mm\nEr: 4.6\nPolygon Isolation: 8mil/0.2032mm\nRF Trace Width: 13.74mil/0.349mm\nhttps://chemandy.com/calculators/coplanar-waveguide-with-ground-calculator.htm"
+		(exclude_from_sim no)
+		(at 328.93 196.85 0)
+		(effects
+			(font
+				(size 1.27 1.27)
+			)
+			(justify left bottom)
+		)
+	)
+	(text "I²C pins have internal \n2.2k pull-ups."
+		(exclude_from_sim no)
+		(at 369.57 55.88 0)
+		(effects
+			(font
+				(size 1.5 1.5)
+			)
+		)
+	)
+	(text "Locking JST"
+		(exclude_from_sim no)
+		(at 160.02 199.39 0)
+		(effects
+			(font
+				(size 3 3)
+			)
+		)
+	)
+	(text "BlueSMiRF"
+		(exclude_from_sim no)
+		(at 130.81 233.68 0)
+		(effects
+			(font
+				(size 1.27 1.27)
+			)
+			(justify left bottom)
+		)
+	)
+	(text "Power\n"
+		(exclude_from_sim no)
+		(at 169.418 44.704 0)
+		(effects
+			(font
+				(size 3 3)
+			)
+		)
+	)
+	(text "RF Connectors"
+		(exclude_from_sim no)
+		(at 360.68 120.65 0)
+		(effects
+			(font
+				(size 3 3)
+			)
+		)
+	)
+	(text "LEDs\n"
+		(exclude_from_sim no)
+		(at 255.27 198.12 0)
+		(effects
+			(font
+				(size 3 3)
+			)
+		)
+	)
+	(text "LG580P Quadband GNSS Receiver"
+		(exclude_from_sim no)
+		(at 326.39 24.13 0)
+		(effects
+			(font
+				(size 3 3)
+			)
+		)
+	)
+	(text "USB to Serial"
+		(exclude_from_sim no)
+		(at 47.752 23.114 0)
+		(effects
+			(font
+				(size 3 3)
+			)
+		)
+	)
+	(text "Battery Backup"
+		(exclude_from_sim no)
+		(at 255.27 134.62 0)
+		(effects
+			(font
+				(size 3 3)
+			)
+		)
+	)
+	(text "SPI interface not yet supported.\nSupport coming in future firmware release."
+		(exclude_from_sim no)
+		(at 368.3 101.6 0)
+		(effects
+			(font
+				(size 3 3)
+			)
+		)
+	)
+	(text "External PTH Connectors"
+		(exclude_from_sim no)
+		(at 72.39 199.39 0)
+		(effects
+			(font
+				(size 3 3)
+			)
+		)
+	)
+	(text "No external I²C pull-ups because \nLG580P has internal resistors."
+		(exclude_from_sim no)
+		(at 175.26 142.24 0)
+		(effects
+			(font
+				(size 1.5 1.5)
+			)
+		)
+	)
 	(junction
 		(at 389.89 142.24)
@@
 		)
 	)
-	(text "I²C Connectors"
-		(exclude_from_sim no)
-		(at 105.41 124.46 0)
-		(effects
-			(font
-				(size 3 3)
-			)
-		)
-	)
-	(text "Generally speaking the ports are used as follows:\nUART1 - Configure in and NMEA output over USB\nUART2 - RTCM correction input and NMEA output over Bluetooth\nUART3 - NMEA output to embedded system"
-		(exclude_from_sim no)
-		(at 116.84 254 0)
-		(effects
-			(font
-				(size 1.5 1.5)
-			)
-			(justify left)
-		)
-	)
-	(text "Reset has\ninternal pull-up."
-		(exclude_from_sim no)
-		(at 289.56 41.91 0)
-		(effects
-			(font
-				(size 1.5 1.5)
-			)
-		)
-	)
-	(text "I²C interface not yet supported.\nSupport coming in future firmware release."
-		(exclude_from_sim no)
-		(at 101.6 163.83 0)
-		(effects
-			(font
-				(size 3 3)
-			)
-		)
-	)
-	(text "Coplanar 50Ω Waveguide Calculation:\nCopper Thickness (1oz): 1.4mil/0.035mm\nBoard thickness: 1.6mm\nDielectric thickness (layer 1 to 2): 0.2mm\nEr: 4.6\nPolygon Isolation: 8mil/0.2032mm\nRF Trace Width: 13.74mil/0.349mm\nhttps://chemandy.com/calculators/coplanar-waveguide-with-ground-calculator.htm"
-		(exclude_from_sim no)
-		(at 328.93 196.85 0)
-		(effects
-			(font
-				(size 1.27 1.27)
-			)
-			(justify left bottom)
-		)
-	)
-	(text "I²C pins have internal \n2.2k pull-ups."
-		(exclude_from_sim no)
-		(at 369.57 55.88 0)
-		(effects
-			(font
-				(size 1.5 1.5)
-			)
-		)
-	)
-	(text "Locking JST"
-		(exclude_from_sim no)
-		(at 160.02 199.39 0)
-		(effects
-			(font
-				(size 3 3)
-			)
-		)
-	)
-	(text "BlueSMiRF"
-		(exclude_from_sim no)
-		(at 130.81 233.68 0)
-		(effects
-			(font
-				(size 1.27 1.27)
-			)
-			(justify left bottom)
-		)
-	)
-	(text "Power\n"
-		(exclude_from_sim no)
-		(at 169.418 44.704 0)
-		(effects
-			(font
-				(size 3 3)
-			)
-		)
-	)
-	(text "RF Connectors"
-		(exclude_from_sim no)
-		(at 360.68 120.65 0)
-		(effects
-			(font
-				(size 3 3)
-			)
-		)
-	)
-	(text "LEDs\n"
-		(exclude_from_sim no)
-		(at 255.27 198.12 0)
-		(effects
-			(font
-				(size 3 3)
-			)
-		)
-	)
-	(text "LG580P Quadband GNSS Receiver"
-		(exclude_from_sim no)
-		(at 326.39 24.13 0)
-		(effects
-			(font
-				(size 3 3)
-			)
-		)
-	)
-	(text "USB to Serial"
-		(exclude_from_sim no)
-		(at 47.752 23.114 0)
-		(effects
-			(font
-				(size 3 3)
-			)
-		)
-	)
-	(text "Battery Backup"
-		(exclude_from_sim no)
-		(at 255.27 134.62 0)
-		(effects
-			(font
-				(size 3 3)
-			)
-		)
-	)
-	(text "SPI interface not yet supported.\nSupport coming in future firmware release."
-		(exclude_from_sim no)
-		(at 368.3 101.6 0)
-		(effects
-			(font
-				(size 3 3)
-			)
-		)
-	)
-	(text "External PTH Connectors"
-		(exclude_from_sim no)
-		(at 72.39 199.39 0)
-		(effects
-			(font
-				(size 3 3)
-			)
-		)
-	)
-	(text "No external I²C pull-ups because \nLG580P has internal resistors."
-		(exclude_from_sim no)
-		(at 175.26 142.24 0)
-		(effects
-			(font
-				(size 1.5 1.5)
-			)
-		)
-	)
 	(global_label "RXD2"
 		(shape input)
@@
 		)
 	)
+	(embedded_fonts no)
 )
